File: KiCad/shop vac controller.kicad_sch (KiCad schematic)
At the start: 32 parts, among them J1 Conn_01x05_Socket, J2 Conn_01x05_Socket, J3 Screw_Terminal_01x02, K1 SSR-20DA, Q1 BS170, U1 CA3140

Commit message: KiCAD update
Other:
- note added: "During initialization the LED's cycle once in one second steps. A solid Red LED indicates that the unit is ready. The Green LED indicates that a trigger from a mains powered tool has been detected. The Blue LED indicates that a trigger from the remote fob has been detected. The Yellow LED indicates the state of the vacuum relay. Solid indicates that the relay is closed, flashing indicates that a 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"
- note removed: "During initialization the LED's cycle once in 1 second steps. A solid Red LED indicates that the unit is ready. The Green LED indicates that a trigger from a mains powered tool has been detected. The Blue LED indicates that a trigger from the remote fob has been detected. The Yellow LED indicates the state of the vacuum relay. Solid indicates that the relay is closed, flashing indicates that a "w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"
Changed lines of the file:
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@@
 		)
 	)
-	(text "During initialization the LED's cycle once in 1 second steps.\n\nA solid Red LED indicates that the unit is ready.\n\nThe Green LED indicates that a trigger from a mains powered tool has been detected.\n\nThe Blue LED indicates that a trigger from the remote fob has been detected.\n\nThe Yellow LED indicates the state of the vacuum relay. Solid indicates that the relay is closed, flashing indicates that a \"wait\" is in progress.\n\nWhen the unit is triggered by a mains powered tool starting it flashes indicating that a 3s delay is in progress before starting the vacuuum.\nThis reduces the additional power surge of both the vacuum and the tool starting together.\n\nThe trigger sensitivity for the power tool is adjusted using RV1.\n\nWhen the unit detects that the that the vacuum is no longer required it flashes the Yellow LED indicating that an adjustable \"shutdown\" period\nhas been initiated allowing dust extraction from the vacuum hose.\n\nThis period is adjustable between 3s and 30s using the potentiometer RV2."
+	(text "During initialization the LED's cycle once in one second steps.\n\nA solid Red LED indicates that the unit is ready.\n\nThe Green LED indicates that a trigger from a mains powered tool has been detected.\n\nThe Blue LED indicates that a trigger from the remote fob has been detected.\n\nThe Yellow LED indicates the state of the vacuum relay. Solid indicates that the relay is closed, flashing indicates that a \"wait\" is in progress.\n\nWhen the unit is triggered by a mains powered tool starting it flashes indicating that a 3s delay is in progress before starting the vacuuum.\nThis reduces the additional power surge of both the vacuum and the tool starting together.\n\nThe trigger sensitivity for the power tool is adjusted using RV1.\n\nWhen the unit detects that the that the vacuum is no longer required it flashes the Yellow LED indicating that an adjustable \"shutdown\" period\nhas been initiated allowing dust extraction from the vacuum hose.\n\nThis period is adjustable between 3s and 30s using the potentiometer RV2."
 		(exclude_from_sim no)
 		(at 33.02 234.95 0)
